Commit message: rsp fixed

File: rb1_ros2_description/urdf/common.gazebo.xacro (robot description, xacro)
@@ -2,6 +2,12 @@
 <robot xmlns:xacro="http://www.ros.org/wiki/xacro">
 	<!-- ROS CONTROL GAZEBO PLUGIN -->
-    <!-- <xacro:macro name="ros2_control">
-	</xacro:macro> -->
+    <xacro:macro name="ros2_control_gazebo">
+        <gazebo>
+            <plugin filename="libgazebo_ros2_control.so" name="gazebo_ros2_control">
+                <robot_param_node>/rb1_robot/robot_state_publisher</robot_param_node>
+                <parameters>$(find rb1_ros2_description)/config/rb1_controller.yaml</parameters>
+            </plugin>
+        </gazebo>
+	</xacro:macro>
 	<xacro:macro name="gazebo_colors" params="prefix">
 		<gazebo reference="$(arg prefix)base_footprint">

File: rb1_ros2_description/urdf/elevator/elevator.gazebo.xacro (robot description, xacro)
@@ -8,5 +8,5 @@
 			<kd value="1.0" />
 			<fdir1 value="1 0 0"/>
-			<material>Gazebo/Grey</material>
+			<material>Gazebo/Black</material>
 			<turnGravityOff>false</turnGravityOff>
 			<!--kp>500000.0</kp>

File: rb1_ros2_description/urdf/elevator/elevator.urdf.xacro (robot description, xacro)
@@ -6,9 +6,9 @@
 	<!-- name : name of the link: -->
 	<!-- hq: selects model in high quality (.dae) -->
-    <xacro:macro name="solid_cuboid_inertia" params="m h d w">
+    <xacro:macro name="solid_cuboid_inertia1" params="m h d w">
 		<inertia  ixx="${(m*(h*h+d*d))/12}" ixy = "0" ixz = "0"
               iyy="${(m*(w*w+d*d))/12}" iyz = "0"
               izz="${(m*(w*w+h*h))/12}"
-     />
+        />
     </xacro:macro>
 	<!-- ELEVATOR_BASE_LINK -->
@@ -27,7 +27,7 @@
 		</inertial-->
 		<inertial>
-			<mass value="0.005" />
+			<mass value="2" />
 			<origin xyz="0 0 -0.27" />
-			<xacro:solid_cuboid_inertia m="0.005" h="0.05" d="0.05" w="0.05"/>
+			<xacro:solid_cuboid_inertia1 m="2" h="0.05" d="0.05" w="0.05"/>
 		</inertial>
 		<visual>
@@ -43,5 +43,5 @@
 				</geometry>
 			</xacro:unless>
-			<material name="darkgrey">
+			<material name="black">
 				<color rgba="0.1 0.1 0.1 1"/>
 			</material>
@@ -60,5 +60,7 @@
 			<child link="${prefix}_platform_link" />
 			<axis xyz="0 0 1"/>
-			<limit effort="10.0" lower="0.0" upper="0.034" velocity="0.5"/>
+			<limit effort="1000.0" lower="0.0" upper="0.034" velocity="0.05"/>
+            <dynamics damping="0.9" friction="1.0"/>
+            <!-- upper="0.034 -->
 	</joint>
 	<link name="${prefix}_platform_link">
@@ -69,7 +71,8 @@
 		</inertial-->
 		<inertial>
-			<mass value="0.005" />
+			<mass value="2" />
 			<origin xyz="0 0 -0.27" />
-			<xacro:solid_cuboid_inertia m="0.005" h="0.05" d="0.05" w="0.05"/>
+			<!-- <solid_cuboid_inertia m="0.005" h="0.05" d="0.05" w="0.05"/> -->
+            <xacro:solid_cuboid_inertia1 m="2" h="0.05" d="0.05" w="0.05"/>
 		</inertial>
 		<visual>
@@ -91,4 +94,5 @@
 		<collision>
 			<origin xyz="0 0 0" rpy="0 0 0 " />
+			<mass>2</mass>
 			<geometry>
 				<mesh filename="package://rb1_ros2_description/meshes/elevator/rb1_elevator_platform.dae"/>

File: rb1_ros2_description/urdf/hokuyo_ust20lx.urdf.xacro (robot description, xacro)
@@ -17,5 +17,5 @@
         <origin xyz="0 0 0.0" rpy="0 0 0"/>
         <geometry>
-            <mesh filename="package://rb1_ros2_description/meshes/hokuyo_ust_20lx.dae"/>
+            <mesh filename="package://rb1_ros2_description/meshes/sensors/hokuyo/hokuyo_ust_20lx.dae"/>
         </geometry>
       </visual>
@@ -26,16 +26,16 @@
       </inertial>
     </link>
-    <link name="${prefix}_link">
-	</link>
+    <!-- <link name="${prefix}_link">
+	  </link>
     <joint name="${prefix}_joint" type="fixed">
       <parent link="${prefix}_base_link"/>
       <child link="${prefix}_link"/>
       <origin xyz="0.00 0.0 0.0474" rpy="0 0 0"/>
-	</joint>
+	  </joint> -->
     <!-- Hokuyo sensor for simulation -->
     <xacro:sensor_hokuyo_ust20_gazebo/>
   </xacro:macro>
   <xacro:macro name="sensor_hokuyo_ust20_gazebo">
-    <gazebo reference="${prefix}_link">
+    <gazebo reference="${prefix}_front_laser_link">
 			<xacro:if value="${gpu}">
         <xacro:property name="ray_type" value="gpu_ray" />
@@ -43,38 +43,41 @@
       </xacro:if>
       <xacro:unless value="${gpu}">
-        <xacro:property name="ray_type" value="ray" />
-        <xacro:property name="plugin_lib" value="libgazebo_ros_laser.so" />
+        <xacro:property name="type" value="ray" />
+        <xacro:property name="plugin_lib" value="libgazebo_ros_ray_laser.so" />
       </xacro:unless>
-			<sensor type="${ray_type}" name="${prefix}_sensor">
-				<pose>0 0 0 0 0 0</pose>
-				<visualize>false</visualize>
-				<update_rate>40</update_rate>
-				<ray>
-					<scan>
-						<horizontal>
-							<samples>1081</samples>
-							<resolution>1</resolution>
-							<min_angle>${min_angle}</min_angle>
-							<max_angle>${max_angle}</max_angle>
-						</horizontal>
-					</scan>
-					<range>
-						<min>0.06</min>
-						<max>20.0</max>
-						<!-- resolution>0.004363323</resolution -->
-						<resolution>0.004359297</resolution>
-						<!-- resolution>0.001</resolution -->
-					</range>
-					<noise>
-						<type>gaussian</type>
-						<mean>0.0</mean>
-						<stddev>0.01</stddev>
-					</noise>
-				</ray>
-				<plugin name="${prefix}_controller" filename="${plugin_lib}">
-					<topicName>${prefix_topic}/scan</topicName>
-					<frameName>/${prefix}_link</frameName>
-				</plugin>
-			</sensor>
+        <sensor type="${type}" name="lidar">
+            <always_on>true</always_on>
+            <visualize>false</visualize>
+            <update_rate>20</update_rate>
+            <ray>
+                <scan>
+                    <horizontal>
+                        <samples>1081</samples>
+                        <resolution>1</resolution>
+                        <min_angle>${min_angle}</min_angle>
+                        <max_angle>${max_angle}</max_angle>
+                    </horizontal>
+                </scan>
+                <range>
+                    <min>0.06</min>
+                    <max>20.0</max>
+                    <!-- resolution>0.004363323</resolution -->
+                    <resolution>0.004359297</resolution>
+                    <!-- resolution>0.001</resolution -->
+                </range>
+                <noise>
+                    <type>gaussian</type>
+                    <mean>0.0</mean>
+                    <stddev>0.01</stddev>
+                </noise>
+            </ray>
+            <plugin name="scan" filename="${plugin_lib}">
+            <ros>
+                <remmaping>~/out:=scan</remmaping>
+            </ros>
+            <output_type>sensor_msgs/LaserScan</output_type>
+            <frame_name>rb1_robot/${prefix}_front_laser_link</frame_name>
+            </plugin>
+        </sensor>
 	</gazebo>
   </xacro:macro>

File: rb1_ros2_description/xacro/rb1_ros2_base.urdf.xacro (robot description, xacro)
@@ -34,10 +34,12 @@
 	<xacro:property name="omni_front_y" value="0.1535" />
 	<xacro:property name="omni_front_z" value="0.0270" />
-	<!-- Flag to select the high or low quality model -->
-	<xacro:property name="hq" value="true" />
+    <!-- ******************* -->
 	<!-- ELEVATOR PARAMETERS -->
+	<!-- ******************* -->
 	<xacro:property name="elevator_x" value="0.0" />
 	<xacro:property name="elevator_y" value="0.0" />
 	<xacro:property name="elevator_z" value="0.213" />
+	<!-- Flag to select the high or low quality model -->
+	<xacro:property name="hq" value="true" />
 	<xacro:arg name="prefix" default="robot_"/>
 	<xacro:arg name="ros_planar_move_plugin" default="false"/>
@@ -53,4 +55,8 @@
 	</xacro:if>
 	<xacro:gazebo_colors prefix="$(arg prefix)"/>
+    <!-- Robot Evelator -->
+    <xacro:elevator_platform prefix="$(arg prefix)evelator" parent="$(arg prefix)base_link" hq="${hq}">
+        <origin xyz="${elevator_x} -${elevator_y} ${elevator_z}" rpy="0 0 0"/>
+    </xacro:elevator_platform>
 	<!-- WHEELS -->
 	<xacro:rubber_wheel prefix="$(arg prefix)right" parent="$(arg prefix)base_link" reflect="false" hq="${hq}">
@@ -70,19 +76,89 @@
 		<origin xyz="${omni_front_x} -${omni_front_y} ${omni_front_z}" rpy="0 0 0"/>
 	</xacro:omni_wheel>
-    <!-- ELEVATOR_PLATFORM -->
-	<xacro:elevator_platform prefix="$(arg prefix)elevator" parent="$(arg prefix)base_link" hq="${hq}">
-		<origin xyz="${elevator_x} -${elevator_y} ${elevator_z}" rpy="0 0 0"/>
-	</xacro:elevator_platform>
 	<!-- SENSORS -->
 	<xacro:sensor_hokuyo_ust20lx prefix="$(arg prefix)front_laser" parent="$(arg prefix)base_link" prefix_topic="front_laser" gpu="$(arg gpu)">
 		<origin xyz="0.210 0.0 0.21" rpy="0 3.1416 3.1416"/>
 	</xacro:sensor_hokuyo_ust20lx>
-	<xacro:sensor_imu_hector prefix="$(arg prefix)imu" parent="$(arg prefix)base_link">
+	<!-- <xacro:sensor_imu_hector prefix="$(arg prefix)imu" parent="$(arg prefix)base_link">
 		<origin xyz="0.002 0.053 0.1485" rpy="0 0 0"/>
-	</xacro:sensor_imu_hector>
-	<xacro:sensor_orbbec_astra prefix="$(arg prefix)front_rgbd_camera" parent="$(arg prefix)base_link" prefix_topic="front_rgbd_camera">
+	</xacro:sensor_imu_hector> -->
+	<!-- <xacro:sensor_orbbec_astra prefix="$(arg prefix)front_rgbd_camera" parent="$(arg prefix)base_link" prefix_topic="front_rgbd_camera">
 		<origin xyz="0.234 0.0 0.092" rpy="0 0 0"/>
-	</xacro:sensor_orbbec_astra>
-	<!-- Gazebo ros2 control plugins -->
-	<xacro:include filename="$(find rb1_ros2_description)/urdf/utils/control.xacro" />
+	</xacro:sensor_orbbec_astra> -->
+    <gazebo reference="$(arg prefix)front_laser_base_link">
+        <sensor name="lidar" type="ray">
+          <always_on>true</always_on>
+          <visualize>false</visualize>
+          <update_rate>20</update_rate>
+          <ray>
+              <scan>
+                  <horizontal>
+                  <samples>1081</samples>
+                  <resolution>1.000000</resolution>
+                  <min_angle>-2.3562</min_angle>
+                  <max_angle>2.3562</max_angle>
+                  </horizontal>
+              </scan>
+              <range>
+                  <min>0.06</min>
+                  <max>20.0</max>
+                  <resolution>0.004359297</resolution>
+              </range>
+              <noise>
+                  <type>gaussian</type>
+                  <mean>0.0</mean>
+                  <stddev>0.01</stddev>
+              </noise>
+          </ray>
+          <plugin name="scan" filename="libgazebo_ros_ray_sensor.so">
+              <ros>
+                  <!-- <namespace>${robot_name}</namespace> -->
+                  <remapping>~/out:=scan</remapping>
+              </ros>
+              <output_type>sensor_msgs/LaserScan</output_type>
+              <frame_name>robot_front_laser_base_link</frame_name>
+          </plugin>
+      </sensor>
+    </gazebo>
+    <!-- Gazebo ros2 control plugins -->
+    <xacro:ros2_control_gazebo/>
+    <!-- ROS2 control - diff drive -->
+    <ros2_control name="diff_drive" type="system">
+        <hardware>
+          <plugin>gazebo_ros2_control/GazeboSystem</plugin>
+        </hardware>
+        <joint name="robot_left_wheel_joint">
+            <command_interface name="velocity">
+            <param name="min">-1</param>
+            <param name="max">1</param>
+            </command_interface>
+            <state_interface name="position"/>
+            <state_interface name="velocity"/>
+            <state_interface name="effort"/>
+        </joint>
+        <joint name="robot_right_wheel_joint">
+            <command_interface name="velocity">
+            <param name="min">-1</param>
+            <param name="max">1</param>
+            </command_interface>
+            <state_interface name="position"/>
+            <state_interface name="velocity"/>
+            <state_interface name="effort"/>
+        </joint>
+    </ros2_control>
+    <!-- ROS2 control - position -->
+    <ros2_control name="joint_position" type="system">
+        <hardware>
+            <plugin>gazebo_ros2_control/GazeboSystem</plugin>
+        </hardware>
+        <joint name="robot_evelator_platform_joint">
+            <command_interface name="position">
+                <param name="min">0.0</param>
+                <param name="max">0.3</param>
+            </command_interface>
+            <state_interface name="position"/>
+            <state_interface name="velocity"/>
+            <state_interface name="effort"/>
+        </joint>
+    </ros2_control>
 </robot>
